Commit message: feat(sim): ogre2 GUI on native Ubuntu, lighting and robot colours from the photo
- gui_render_engine:=auto (default): ogre2 on a native install, ogre (v1)
  and MESA_GL_VERSION_OVERRIDE only on WSL2, where they were needed.
- robocup_home: ambient light 1.0 -> 0.45 (scene was flat white), sky,
  matte walls, wooden floor inside the house (visual only, no
  self-shadowing), darker ground outside, start view over the house,
  GUI far clip 25000 -> 300 m.
- robot: silver body, black LiDAR and wheels as in the wiki photo
  (appearance.xacro); the turning wheels now show the mecanum mesh
  (rosorin_body.xacro drops the fixed CAD wheel visuals, keeps their
  mass and collision).

Looks only: RTF 1.0, probe_motion 1.00/1.00/1.00, probe_collision 9/9,
/scan 400 beams with no self-hits, 24 package tests pass.

File: src/rosorin_navigation/urdf/rosorin_sim.urdf.xacro (robot description, xacro)
@@ -3,5 +3,6 @@
   ROSOrin Pro simulation model (Ignition Gazebo Fortress).
   Fixed copy of robot_gazebo/urdf/robot.gazebo.xacro (Hiwonder, V1.0.0 2025-05-29). The robot body
-  (rosorin_description/urdf/rosorin.xacro) is used unchanged. Changes, with the evidence for each
+  (rosorin_body.xacro, a copy of rosorin_description/urdf/rosorin.xacro without the fixed wheel
+  visuals) keeps the CAD masses and collisions. Changes, with the evidence for each
   in docs/wiki_findings/ and test/test_sim_fidelity.py:
   - MecanumDrive uses the wiki constants: wheel_radius 0.04, wheel_separation 0.17706,
@@ -17,12 +18,14 @@
     the centre (retail figure for the Standard kit, the wiki does not give a mass)
   - removed the ign_ros2_control plugin (the URDF has no <ros2_control> tag, see ISSUE-009)
+  - colours of the real robot (appearance.xacro); the turning wheels show the mecanum mesh
 -->
 <robot name="robot" xmlns:xacro="http://ros.org/wiki/xacro">
   <xacro:arg name="sim_ign" default="true"/>
-  <xacro:include filename="$(find rosorin_description)/urdf/rosorin.xacro"/>
+  <xacro:include filename="$(find rosorin_navigation)/urdf/rosorin_body.xacro"/>
   <xacro:include filename="$(find rosorin_navigation)/urdf/wheel.xacro"/>
   <xacro:include filename="$(find rosorin_navigation)/urdf/lidar.gazebo.xacro"/>
   <xacro:include filename="$(find rosorin_navigation)/urdf/camera.gazebo.xacro"/>
   <xacro:include filename="$(find robot_gazebo)/urdf/imu.gazebo.xacro"/>
+  <xacro:include filename="$(find rosorin_navigation)/urdf/appearance.xacro"/>
   <!-- mass the CAD model lacks (battery, controller, arm, screen) -->
   <link name="ballast_link">

File: src/rosorin_navigation/urdf/wheel.xacro (robot description, xacro)
@@ -14,4 +14,6 @@
   - joint damping/friction removed (the velocity command already fixes the wheel speed)
   - removed the malformed kp value "1000000000.0.0" (ignored by the DART engine anyway)
+  - visual: the Hiwonder mecanum wheel mesh (rosorin_description, same 0.04 m radius), so the wheels
+    that turn are the ones on screen; the collision stays a cylinder
 -->
 <robot xmlns:xacro="http://www.ros.org/wiki/xacro">
@@ -20,10 +22,13 @@
   <xacro:property name="WHEEL_MASS" value="0.07" />
   <xacro:property name="WHEEL_MU" value="0.0" />
-  <xacro:macro name="mecanum_wheel" params="name x y">
+  <!-- mesh: CAD wheel mesh; mesh_y: shift that centres it on the axle (the mesh spans y 0..0.038) -->
+  <xacro:macro name="mecanum_wheel" params="name x y mesh mesh_y">
     <link name="${name}_link">
       <visual>
-        <geometry><cylinder radius="${WHEEL_RADIUS}" length="${WHEEL_LENGTH}"/></geometry>
+        <geometry>
+          <mesh filename="file://$(find rosorin_description)/meshes/${mesh}.stl"/>
+        </geometry>
         <material name="black"><color rgba="0 0 0 1"/></material>
-        <origin rpy="1.5707 0 0"/>
+        <origin xyz="0 ${mesh_y} 0"/>
       </visual>
       <collision>
@@ -50,7 +55,11 @@
   </xacro:macro>
   <!-- x: CAD wheel positions (0.090972 / -0.080677); y: +-0.17706 / 2 -->
-  <xacro:mecanum_wheel name="front_left"  x="0.090972"  y="0.08853"/>
-  <xacro:mecanum_wheel name="front_right" x="0.090972"  y="-0.08853"/>
-  <xacro:mecanum_wheel name="rear_left"   x="-0.080677" y="0.08853"/>
-  <xacro:mecanum_wheel name="rear_right"  x="-0.080677" y="-0.08853"/>
+  <xacro:mecanum_wheel name="front_left"  x="0.090972"  y="0.08853"
+                       mesh="left_front_wheel_link" mesh_y="-0.019"/>
+  <xacro:mecanum_wheel name="front_right" x="0.090972"  y="-0.08853"
+                       mesh="right_front_wheel_link" mesh_y="0.019"/>
+  <xacro:mecanum_wheel name="rear_left"   x="-0.080677" y="0.08853"
+                       mesh="left_back_wheel_link" mesh_y="-0.019"/>
+  <xacro:mecanum_wheel name="rear_right"  x="-0.080677" y="-0.08853"
+                       mesh="right_back_wheel_link" mesh_y="0.019"/>
 </robot>
